Commit message: working sim

File: meca500_description/urdf/meca500.gazebo.xacro (robot description, xacro)
@@ -4,5 +4,5 @@
     <!-- gz_ros2_control plugin: starts the embedded controller_manager in Gazebo -->
     <gazebo>
-      <plugin filename="gz_ros2_control-system"
+      <plugin filename="libgz_ros2_control-system.so"
               name="gz_ros2_control::GazeboSimROS2ControlPlugin">
         <parameters>$(find meca500_bringup)/config/meca500_controllers.yaml</parameters>

File: meca500_description/urdf/meca500.ros2_control.xacro (robot description, xacro)
@@ -60,5 +60,5 @@
     <ros2_control name="${name}" type="system">
       <hardware>
-        <plugin>gz_ros2_control/GazeboSystem</plugin>
+        <plugin>gz_ros2_control/GazeboSimSystem</plugin>
       </hardware>
       <joint name="meca_axis_1">

File: meca500_description/urdf/meca500.urdf.xacro (robot description, xacro)
@@ -1,11 +1,17 @@
 <?xml version="1.0"?>
 <robot xmlns:xacro="http://www.ros.org/wiki/xacro" name="Meca500_R4">
-  <xacro:arg name="use_sim_hardware" default="false"/>
+  <xacro:arg name="use_sim_hardware" default="true"/>
   <xacro:arg name="robot_ip"         default="192.168.0.100"/>
   <xacro:include filename="meca500_macro.xacro"/>
   <xacro:include filename="meca500.ros2_control.xacro"/>
   <xacro:include filename="meca500.gazebo.xacro"/>
-  <link name="world"/>
-  <xacro:meca500 parent="world">
+  <!-- Root link for mounting the robot (with minimal inertia for Gazebo) -->
+  <link name="robot_base">
+    <inertial>
+      <mass value="0.001"/>
+      <inertia ixx="0.0001" ixy="0" ixz="0" iyy="0.0001" iyz="0" izz="0.0001"/>
+    </inertial>
+  </link>
+  <xacro:meca500 parent="robot_base">
     <origin xyz="0 0 0" rpy="0 0 0"/>
   </xacro:meca500>

File: meca500_description/urdf/meca500_macro.xacro (robot description, xacro)
@@ -189,6 +189,6 @@
       <inertial>
         <origin xyz="0 0 0" rpy="0 0 0"/>
-        <mass value="0"/>
-        <inertia ixx="0" ixy="0" ixz="0" iyy="0" iyz="0" izz="0"/>
+        <mass value="0.05"/>
+        <inertia ixx="0.0001" ixy="0" ixz="0" iyy="0.0001" iyz="0" izz="0.0001"/>
       </inertial>
       <collision>
