Commit message: Sim Added

File: meca500_description/urdf/meca500.ros2_control.xacro (robot description, xacro)
@@ -57,3 +57,58 @@
     </ros2_control>
   </xacro:macro>
+  <xacro:macro name="meca500_ros2_control_sim" params="name">
+    <ros2_control name="${name}" type="system">
+      <hardware>
+        <plugin>gz_ros2_control/GazeboSystem</plugin>
+      </hardware>
+      <joint name="meca_axis_1">
+        <command_interface name="velocity">
+          <param name="min">-2.61</param>
+          <param name="max">2.61</param>
+        </command_interface>
+        <state_interface name="position"/>
+        <state_interface name="velocity"/>
+      </joint>
+      <joint name="meca_axis_2">
+        <command_interface name="velocity">
+          <param name="min">-2.61</param>
+          <param name="max">2.61</param>
+        </command_interface>
+        <state_interface name="position"/>
+        <state_interface name="velocity"/>
+      </joint>
+      <joint name="meca_axis_3">
+        <command_interface name="velocity">
+          <param name="min">-3.14</param>
+          <param name="max">3.14</param>
+        </command_interface>
+        <state_interface name="position"/>
+        <state_interface name="velocity"/>
+      </joint>
+      <joint name="meca_axis_4">
+        <command_interface name="velocity">
+          <param name="min">-5.23</param>
+          <param name="max">5.23</param>
+        </command_interface>
+        <state_interface name="position"/>
+        <state_interface name="velocity"/>
+      </joint>
+      <joint name="meca_axis_5">
+        <command_interface name="velocity">
+          <param name="min">-5.23</param>
+          <param name="max">5.23</param>
+        </command_interface>
+        <state_interface name="position"/>
+        <state_interface name="velocity"/>
+      </joint>
+      <joint name="meca_axis_6">
+        <command_interface name="velocity">
+          <param name="min">-8.72</param>
+          <param name="max">8.72</param>
+        </command_interface>
+        <state_interface name="position"/>
+        <state_interface name="velocity"/>
+      </joint>
+    </ros2_control>
+  </xacro:macro>
 </robot>

File: meca500_description/urdf/meca500.urdf.xacro (robot description, xacro)
@@ -1,10 +1,19 @@
 <?xml version="1.0"?>
 <robot xmlns:xacro="http://www.ros.org/wiki/xacro" name="Meca500_R4">
+  <xacro:arg name="use_sim_hardware" default="false"/>
+  <xacro:arg name="robot_ip"         default="192.168.0.100"/>
   <xacro:include filename="meca500_macro.xacro"/>
   <xacro:include filename="meca500.ros2_control.xacro"/>
+  <xacro:include filename="meca500.gazebo.xacro"/>
   <link name="world"/>
   <xacro:meca500 parent="world">
     <origin xyz="0 0 0" rpy="0 0 0"/>
   </xacro:meca500>
-  <xacro:meca500_ros2_control name="Meca500System" robot_ip="192.168.0.100"/>
+  <xacro:if value="$(arg use_sim_hardware)">
+    <xacro:meca500_ros2_control_sim name="Meca500System"/>
+    <xacro:meca500_gazebo/>
+  </xacro:if>
+  <xacro:unless value="$(arg use_sim_hardware)">
+    <xacro:meca500_ros2_control name="Meca500System" robot_ip="$(arg robot_ip)"/>
+  </xacro:unless>
 </robot>

Commit message: aasdf

File: meca500_description/urdf/meca500.ros2_control.xacro (robot description, xacro)
@@ -1,5 +1,60 @@
 <?xml version="1.0"?>
 <robot xmlns:xacro="http://www.ros.org/wiki/xacro">
-  <xacro:macro name="meca500_ros2_control" params="name robot_ip">
+  <xacro:include filename="$(find beckhoff_ads_bringup)/urdf/beckhoff_bot/beckhoff_ads_interfaces.ros2_control.xacro"/>
+  <xacro:if value="$(arg sim_mode)">
+    <ros2_control name="${name}" type="system">
+      <hardware>
+        <plugin>gz_ros2_control/GazeboSimSystem</plugin>
+      </hardware>
+      <joint name="meca_axis_1">
+        <command_interface name="velocity">
+          <param name="min">-2.61</param>
+          <param name="max">2.61</param>
+        </command_interface>
+        <state_interface name="position"/>
+        <state_interface name="velocity"/>
+      </joint>
+      <joint name="meca_axis_2">
+        <command_interface name="velocity">
+          <param name="min">-2.61</param>
+          <param name="max">2.61</param>
+        </command_interface>
+        <state_interface name="position"/>
+        <state_interface name="velocity"/>
+      </joint>
+      <joint name="meca_axis_3">
+        <command_interface name="velocity">
+          <param name="min">-3.14</param>
+          <param name="max">3.14</param>
+        </command_interface>
+        <state_interface name="position"/>
+        <state_interface name="velocity"/>
+      </joint>
+      <joint name="meca_axis_4">
+        <command_interface name="velocity">
+          <param name="min">-5.23</param>
+          <param name="max">5.23</param>
+        </command_interface>
+        <state_interface name="position"/>
+        <state_interface name="velocity"/>
+      </joint>
+      <joint name="meca_axis_5">
+        <command_interface name="velocity">
+          <param name="min">-5.23</param>
+          <param name="max">5.23</param>
+        </command_interface>
+        <state_interface name="position"/>
+        <state_interface name="velocity"/>
+      </joint>
+      <joint name="meca_axis_6">
+        <command_interface name="velocity">
+          <param name="min">-8.72</param>
+          <param name="max">8.72</param>
+        </command_interface>
+        <state_interface name="position"/>
+        <state_interface name="velocity"/>
+      </joint>
+    </ros2_control>
+  </xacro:if>
     <ros2_control name="${name}" type="system">
       <hardware>
@@ -56,9 +111,9 @@
       </joint>
     </ros2_control>
-  </xacro:macro>
-  <xacro:macro name="meca500_ros2_control_sim" params="name">
-    <ros2_control name="${name}" type="system">
-      <hardware>
-        <plugin>gz_ros2_control/GazeboSimSystem</plugin>
+  <xacro:if value="$(not sim_mode)">
+    <ros2_control name="${name}" type="system">
+      <hardware>
+        <plugin>meca500_hardware/Meca500SystemHardware</plugin>
+        <param name="robot_ip">${robot_ip}</param>
       </hardware>
       <joint name="meca_axis_1">
@@ -111,4 +166,38 @@
       </joint>
     </ros2_control>
-  </xacro:macro>
+  </xacro:if>
+  <xacro:if value="$(not alone)">
+    <ros2_control name="${name}" type="system">
+      <hardware>
+        <plugin>beckhoff_ads_hardware_interface/BeckhoffADSHardwareInterface</plugin>
+        <param name="plc_ip_address">192.168.122.2</param>
+        <param name="plc_ams_net_id">192.168.122.2.1.1</param>
+        <param name="plc_ams_port">851</param>
+        <param name="local_ams_net_id">192.168.122.1.1.1</param>
+      </hardware>
+    </ros2_control>
+    <gpio name="meca_io">
+          <xacro:command_interface_PLC name="robotEnabled" PLC_symbol="MAIN.robotEnabled" PLC_type="BOOL" initial_value="1"/>
+          <xacro:command_interface_PLC name="robotMode" PLC_symbol="MAIN.robotMode" PLC_type="UDINT" initial_value="1"/>
+          <xacro:command_interface_PLC name="joint_1_cmd" PLC_symbol="MAIN.jointCommands" PLC_type="LREAL" n_elements="6" index="0" initial_value="0.0"/>
+          <xacro:command_interface_PLC name="joint_2_cmd" PLC_symbol="MAIN.jointCommands" PLC_type="LREAL" n_elements="6" index="1" initial_value="0.0"/>
+          <xacro:command_interface_PLC name="joint_3_cmd" PLC_symbol="MAIN.jointCommands" PLC_type="LREAL" n_elements="6" index="2" initial_value="0.0"/>
+          <xacro:command_interface_PLC name="joint_4_cmd" PLC_symbol="MAIN.jointCommands" PLC_type="LREAL" n_elements="6" index="3" initial_value="0.0"/>
+          <xacro:command_interface_PLC name="joint_5_cmd" PLC_symbol="MAIN.jointCommands" PLC_type="LREAL" n_elements="6" index="4" initial_value="0.0"/>
+          <xacro:command_interface_PLC name="joint_6_cmd" PLC_symbol="MAIN.jointCommands" PLC_type="LREAL" n_elements="6" index="5" initial_value="0.0"/>
+        </gpio>
+        <sensor name="meca_sensor">
+          <xacro:state_interface_PLC name="robotStatus" PLC_symbol="MAIN.robotStatus" PLC_type="UDINT"/>
+          <xacro:state_interface_PLC name="robotError" PLC_symbol="MAIN.robotError" PLC_type="BOOL"/>
+          <xacro:state_interface_PLC name="joint_1_state" PLC_symbol="MAIN.jointStates" PLC_type="LREAL" n_elements="6" index="0"/>
+          <xacro:state_interface_PLC name="joint_2_state" PLC_symbol="MAIN.jointStates" PLC_type="LREAL" n_elements="6" index="1"/>
+          <xacro:state_interface_PLC name="joint_3_state" PLC_symbol="MAIN.jointStates" PLC_type="LREAL" n_elements="6" index="2"/>
+          <xacro:state_interface_PLC name="joint_4_state" PLC_symbol="MAIN.jointStates" PLC_type="LREAL" n_elements="6" index="3"/>
+          <xacro:state_interface_PLC name="joint_5_state" PLC_symbol="MAIN.jointStates" PLC_type="LREAL" n_elements="6" index="4"/>
+          <xacro:state_interface_PLC name="joint_6_state" PLC_symbol="MAIN.jointStates" PLC_type="LREAL" n_elements="6" index="5"/>
+          <!-- Mirror command interfaces for monitoring -->
+          <xacro:state_interface_PLC name="robotEnabled" PLC_symbol="MAIN.robotEnabled" PLC_type="BOOL"/>
+          <xacro:state_interface_PLC name="robotMode" PLC_symbol="MAIN.robotMode" PLC_type="UDINT"/>
+        </sensor>
+  </xacro:if>
 </robot>

File: meca500_description/urdf/meca500.urdf.xacro (robot description, xacro)
@@ -1,6 +1,8 @@
 <?xml version="1.0"?>
 <robot xmlns:xacro="http://www.ros.org/wiki/xacro" name="Meca500_R4">
-  <xacro:arg name="use_sim_hardware" default="true"/>
   <xacro:arg name="robot_ip"         default="192.168.0.100"/>
+  <xacro:arg name="sim_mode"         default="false"/>
+  <xacro:arg name="alone"            default="true"/>
+  <xacro:arg name="name"             default="DummyBot"/>
   <xacro:include filename="meca500_macro.xacro"/>
   <xacro:include filename="meca500.ros2_control.xacro"/>
@@ -16,10 +18,9 @@
     <origin xyz="0 0 0" rpy="0 0 0"/>
   </xacro:meca500>
-  <xacro:if value="$(arg use_sim_hardware)">
-    <xacro:meca500_ros2_control_sim name="Meca500System"/>
+  <!-- Unified ros2_control macro -->
+  <xacro:meca500_ros2_control name="Meca500System" robot_ip="$(arg robot_ip)" sim_mode="$(arg sim_mode)" alone="$(arg alone)"/>
+  <!-- Include Gazebo plugin if in sim mode -->
+  <xacro:if value="$(arg sim_mode)">
     <xacro:meca500_gazebo/>
   </xacro:if>
-  <xacro:unless value="$(arg use_sim_hardware)">
-    <xacro:meca500_ros2_control name="Meca500System" robot_ip="$(arg robot_ip)"/>
-  </xacro:unless>
 </robot>
