Commit message: Working Sim Mode and seperate beckhoff

File: meca500_description/urdf/meca500.gazebo.macro.xacro (robot description, xacro)
@@ -2,9 +2,8 @@
 <robot xmlns:xacro="http://www.ros.org/wiki/xacro">
   <xacro:macro name="meca500_gazebo">
-    <!-- gz_ros2_control plugin: starts the embedded controller_manager in Gazebo -->
     <gazebo>
-      <plugin filename="libgz_ros2_control-system.so"
-              name="gz_ros2_control::GazeboSimROS2ControlPlugin">
+      <plugin filename="libgz_ros2_control-system.so" name="gz_ros2_control::GazeboSimROS2ControlPlugin">
         <parameters>$(find meca500_bringup)/config/meca500_controllers.yaml</parameters>
+        <controller_manager_name>sim_controller_manager</controller_manager_name>
         <ros>
           <remapping>~/robot_description:=robot_description</remapping>
@@ -40,5 +39,4 @@
       <selfCollide>false</selfCollide>
     </gazebo>
-    <!-- Light damping on each joint prevents oscillation under velocity control -->
     <gazebo reference="meca_axis_1">
       <implicitSpringDamper>true</implicitSpringDamper>

File: meca500_description/urdf/meca500.urdf.xacro (robot description, xacro)
@@ -1,12 +1,11 @@
 <?xml version="1.0"?>
 <robot xmlns:xacro="http://www.ros.org/wiki/xacro" name="Meca500_R4">
-  <xacro:arg name="robot_ip"         default="192.168.0.100"/>
-  <xacro:arg name="sim_mode"         default="false"/>
-  <xacro:arg name="alone"            default="true"/>
-  <xacro:arg name="name"             default="DummyBot"/>
-  <xacro:include filename="meca500_macro.xacro"/>
-  <xacro:include filename="meca500.ros2_control.xacro"/>
-  <xacro:include filename="meca500.gazebo.xacro"/>
-  <!-- Root link for mounting the robot (with minimal inertia for Gazebo) -->
+  <xacro:arg name="robot_ip" default="192.168.0.100"/>
+  <xacro:arg name="sim_mode" default="true"/>
+  <xacro:arg name="name" default="DummyBot"/>
+  <xacro:arg name="alone" default="false"/>
+  <xacro:include filename="meca500_description.macro.xacro"/>
+  <xacro:include filename="meca500.ros2_control.macro.xacro"/>
+  <xacro:include filename="meca500.gazebo.macro.xacro"/>
   <link name="robot_base">
     <inertial>
@@ -15,12 +14,11 @@
     </inertial>
   </link>
-  <xacro:meca500 parent="robot_base">
+  <!-- Description -->
+  <xacro:meca500_descrip parent="robot_base">
     <origin xyz="0 0 0" rpy="0 0 0"/>
-  </xacro:meca500>
-  <!-- Unified ros2_control macro -->
-  <xacro:meca500_ros2_control name="Meca500System" robot_ip="$(arg robot_ip)" sim_mode="$(arg sim_mode)" alone="$(arg alone)"/>
-  <!-- Include Gazebo plugin if in sim mode -->
-  <xacro:if value="$(arg sim_mode)">
-    <xacro:meca500_gazebo/>
-  </xacro:if>
+  </xacro:meca500_descrip>
+  <!-- Control -->
+  <xacro:meca500_ros2_control name="$(arg name)" robot_ip="$(arg robot_ip)" sim_mode="$(arg sim_mode)"/>
+  <!-- Gz -->
+  <xacro:meca500_gazebo/>
 </robot>

File: meca500_description/urdf/meca500_description.macro.xacro (robot description, xacro)
@@ -1,5 +1,5 @@
 <?xml version="1.0"?>
 <robot xmlns:xacro="http://www.ros.org/wiki/xacro">
-  <xacro:macro name="meca500" params="parent *origin">
+  <xacro:macro name="meca500_descrip" params="parent *origin">
     <material name="grey">
       <color rgba="0.2 0.2 0.2 1.0"/>
